File: aout.kicad_sch (KiCad schematic)
At the start: 104 parts, among them J301 OUTPUT1-4, J302 OUTPUT5-8, U301 OPA4134UA, U302 OPA4134UA

Commit message: Cleaned up schematic
Connections:
- net GNDA renamed GND
Changed lines of the file:
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@@
 			)
 		)
-		(property "Value" "GNDA"
+		(property "Value" "GND"
 			(at 57.15 218.44 0)
 			(effects
@@
 			)
 		)
-		(property "Value" "GNDA"
+		(property "Value" "GND"
 			(at 156.21 124.46 0)
 			(effects
@@
 			)
 		)
-		(property "Value" "GNDA"
+		(property "Value" "GND"
 			(at 172.72 215.9 0)
 			(effects
@@
 			)
 		)
-		(property "Value" "GNDA"
+		(property "Value" "GND"
 			(at 323.85 180.34 0)
 			(effects
@@
 			)
 		)
-		(property "Value" "GNDA"
+		(property "Value" "GND"
 			(at 240.03 124.46 0)
 			(effects
@@
 			)
 		)
-		(property "Value" "GNDA"
+		(property "Value" "GND"
 			(at 72.39 181.61 0)
 			(effects
@@
 			)
 		)
-		(property "Value" "GNDA"
+		(property "Value" "GND"
 			(at 88.9 181.61 0)
 			(effects
@@
 			)
 		)
-		(property "Value" "GNDA"
+		(property "Value" "GND"
 			(at 114.3 218.44 0)
 			(effects
@@
 			)
 		)
-		(property "Value" "GNDA"
+		(property "Value" "GND"
 			(at 88.9 124.46 0)
 			(effects
@@
 			)
 		)
-		(property "Value" "GNDA"
+		(property "Value" "GND"
 			(at 172.72 124.46 0)
 			(effects
@@
 			)
 		)
-		(property "Value" "GNDA"
+		(property "Value" "GND"
 			(at 256.54 181.61 0)
 			(effects
@@
 			)
 		)
-		(property "Value" "GNDA"
+		(property "Value" "GND"
 			(at 172.72 180.34 0)
 			(effects
@@
 			)
 		)
-		(property "Value" "GNDA"
+		(property "Value" "GND"
 			(at 204.47 215.9 0)
 			(effects
@@
 			)
 		)
-		(property "Value" "GNDA"
+		(property "Value" "GND"
 			(at 256.54 124.46 0)
 			(effects
@@
 			)
 		)
-		(property "Value" "GNDA"
+		(property "Value" "GND"
 			(at 323.85 124.46 0)
 			(effects
@@
 			)
 		)
-		(property "Value" "GNDA"
+		(property "Value" "GND"
 			(at 156.21 180.34 0)
 			(effects
@@
 			)
 		)
-		(property "Value" "GNDA"
+		(property "Value" "GND"
 			(at 340.36 180.34 0)
 			(effects
@@
 			)
 		)
-		(property "Value" "GNDA"
+		(property "Value" "GND"
 			(at 240.03 181.61 0)
 			(effects
@@
 			)
 		)
-		(property "Value" "GNDA"
+		(property "Value" "GND"
 			(at 72.39 124.46 0)
 			(effects
@@
 			)
 		)
-		(property "Value" "GNDA"
+		(property "Value" "GND"
 			(at 340.36 124.46 0)
 			(effects
